File: Gen 3 Leaf Adapter.kicad_sch (KiCad schematic)
At the start: 89 parts, among them J1 Conn_02x16_Top_Bottom_Mountin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, J2 Conn_02x20_Top_Bottom_Mountin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, J3 Conn_02x05_Odd_Even, J4 Conn_01x06_Male, J8 Conn_01x03_Male, Q1 Q_NMOS_GDS, Q2 Q_NMOS_GDS, Q3 IRLML0100TRPBF, Q4 IRLML0100TRPBF, Q5 IRLML0100TRPBF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

Commit message: V0.0.2
Removed R17, corrected throttle voltages from 0-3.3 to 0-6.6v, corrected schematic notes, mini mainboard symbol (V2), updated silkscreen to V0.0.2, and added a 2nd page to the schematic to track revision changes.
Parts:
- removed R17: 10K, Resistor_SMD:R_0805_2012Metric_Pad1.20x1.40mm_HandSolder, symbol Device:R
Connections:
- net SIG_EMCYSTOP: now also J2.40 (Pin_40), SJ5.2 (B)
Other:
- added sheet Revisions (Revisions.kicad_sch)
- note added: "* = 12V Signal ° = 0-6.6V Signal □ = Switched - ▲ = Switched +12v"
- note removed: "* = 12V Signal ° = 0-3.3V Signal □ = Switched - ▲ = Switched +12v"
- note removed: "~10ms debounce"
Changed lines of the file:
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@@
     (title "Gen 3 Nissan Leaf Mini Mainboard Adapter")
     (date "2023-10-05")
-    (rev "V0.0.1")
+    (rev "V0.0.2")
   )
   (junction (at 43.18 180.34) (diameter 0) (color 0 0 0 0)
@@
     (stroke (width 0) (type default) (color 0 0 0 0))
   )
-  (wire (pts (xy 182.88 85.09) (xy 186.69 85.09))
-    (stroke (width 0) (type default) (color 0 0 0 0))
-  )
   (wire (pts (xy 99.06 25.4) (xy 102.87 25.4))
     (stroke (width 0) (type default) (color 0 0 0 0))
@@
     (stroke (width 0) (type default) (color 0 0 0 0))
   )
-  (wire (pts (xy 194.31 85.09) (xy 198.12 85.09))
+  (wire (pts (xy 182.88 85.09) (xy 198.12 85.09))
     (stroke (width 0) (type default) (color 0 0 0 0))
   )
@@
     (effects (font (size 1.27 1.27)) (justify left bottom))
   )
-  (text "* = 12V Signal\n° = 0-3.3V Signal\n□ = Switched -\n▲ = Switched +12v"
+  (text "* = 12V Signal\n° = 0-6.6V Signal\n□ = Switched -\n▲ = Switched +12v"
     (at 179.07 180.34 0)
     (effects (font (size 2 2)) (justify left bottom))
@@
     (effects (font (size 1.27 1.27)) (justify left bottom))
   )
-  (text "~10ms debounce" (at 195.58 83.82 0)
-    (effects (font (size 1.27 1.27)) (justify left bottom))
-  )
   (text "*" (at 191.77 45.72 0)
     (effects (font (size 1.27 1.27)) (justify left bottom))
@@
     (pin "1")
   )
-  (symbol (lib_id "Device:R") (at 190.5 85.09 270) (unit 1)
-    (in_bom yes) (on_board yes)
-    (property "Reference" "R17" (id 0) (at 187.96 82.55 90))
-    (property "Value" "10K" (id 1) (at 193.04 82.55 90))
-    (property "Footprint" "Resistor_SMD:R_0805_2012Metric_Pad1.20x1.40mm_HandSolder" (id 2) (at 190.5 83.312 90)
-      (effects (font (size 1.27 1.27)) hide)
-    )
-    (property "Datasheet" "~" (id 3) (at 190.5 85.09 0)
-      (effects (font (size 1.27 1.27)) hide)
-    )
-    (property "LCSC Part" "C17414" (id 4) (at 190.5 85.09 0)
-      (effects (font (size 1.27 1.27)) hide)
-    )
-    (property "MFG Part #" "0805W8F1002T5E" (id 5) (at 190.5 85.09 0)
-      (effects (font (size 1.27 1.27)) hide)
-    )
-    (property "Manufacturer" "UNI-ROYAL" (id 6) (at 190.5 85.09 0)
-      (effects (font (size 1.27 1.27)) hide)
-    )
-    (pin "1")
-    (pin "2")
-  )
   (symbol (lib_id "power:GND") (at 246.38 72.39 0) (unit 1)
     (in_bom yes) (on_board yes)
@@
     (pin "2")
   )
+  (sheet (at 257.81 170.18) (size 12.7 7.62) (fields_autoplaced)
+    (stroke (width 0.1524) (type solid) (color 0 0 0 0))
+    (fill (color 0 0 0 0.0000))
+    (property "Sheet name" "Revisions" (id 0) (at 257.81 169.4684 0)
+      (effects (font (size 1.27 1.27)) (justify left bottom))
+    )
+    (property "Sheet file" "Revisions.kicad_sch" (id 1) (at 257.81 178.3846 0)
+      (effects (font (size 1.27 1.27)) (justify left top))
+    )
+  )
   (sheet_instances
     (path "/" (page "1"))
+    (path "/a0459ab7-2e7d-4701-b75f-648acc71baed" (page "2"))
   )
   (symbol_instances
@@
       (reference "R16") (unit 1) (value "10K") (footprint "Resistor_SMD:R_0805_2012Metric_Pad1.20x1.40mm_HandSolder")
     )
-    (path "/25b84e25-487f-4ba6-a1ca-12592879b4df"
-      (reference "R17") (unit 1) (value "10K") (footprint "Resistor_SMD:R_0805_2012Metric_Pad1.20x1.40mm_HandSolder")
-    )
     (path "/d95b4734-69db-4953-a9c4-ed95ea84ced4"

Commit message: V0.0.3 update
Corrected L2 inductor to one properly sized.  From 0805 to a Sunlord 4030 / 4.0mmX4.0mm inductor.
Parts:
- L2: value 10uH 1.15OHM -> 10uH; footprint Inductor_SMD:L_0805_2012Metric_Pad1.15x1.40mm_HandSolder -> OpenInverter Library:Inductor_Sunlord_4030; LCSC Part C1046 -> C38117; MFG Part # SDFL2012S100KTF -> SWPA4030S100MT; Specs (none) -> 10uH, 700ma or +
Changed lines of the file:
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@@
     (title "Gen 3 Nissan Leaf Mini Mainboard Adapter")
     (date "2023-10-05")
-    (rev "V0.0.2")
+    (rev "V0.0.3")
   )
   (junction (at 43.18 180.34) (diameter 0) (color 0 0 0 0)
@@
     (in_bom yes) (on_board yes)
     (property "Reference" "L2" (id 0) (at 35.56 175.514 90))
-    (property "Value" "10uH 1.15OHM" (id 1) (at 35.56 177.8254 90))
-    (property "Footprint" "Inductor_SMD:L_0805_2012Metric_Pad1.15x1.40mm_HandSolder" (id 2) (at 35.56 180.34 0)
+    (property "Value" "10uH" (id 1) (at 35.56 177.8254 90))
+    (property "Footprint" "OpenInverter Library:Inductor_Sunlord_4030" (id 2) (at 35.56 180.34 0)
       (effects (font (size 1.27 1.27)) hide)
     )
@@
       (effects (font (size 1.27 1.27)) hide)
     )
-    (property "LCSC Part" "C1046" (id 4) (at 35.56 180.34 0)
+    (property "Manufacturer" "SUNLORD" (id 6) (at 35.56 180.34 0)
       (effects (font (size 1.27 1.27)) hide)
     )
-    (property "MFG Part #" "SDFL2012S100KTF" (id 5) (at 35.56 180.34 0)
+    (property "LCSC Part" "C38117" (id 7) (at 35.56 180.34 0)
       (effects (font (size 1.27 1.27)) hide)
     )
-    (property "Manufacturer" "SUNLORD" (id 6) (at 35.56 180.34 0)
+    (property "MFG Part #" "SWPA4030S100MT" (id 8) (at 35.56 180.34 0)
+      (effects (font (size 1.27 1.27)) hide)
+    )
+    (property "Specs" "10uH, 700ma or +" (id 9) (at 35.56 180.34 0)
       (effects (font (size 1.27 1.27)) hide)
     )
@@
     )
     (path "/79d88cca-9340-4019-9ee8-122b367e6acf"
-      (reference "L2") (unit 1) (value "10uH 1.15OHM") (footprint "Inductor_SMD:L_0805_2012Metric_Pad1.15x1.40mm_HandSolder")
+      (reference "L2") (unit 1) (value "10uH") (footprint "OpenInverter Library:Inductor_Sunlord_4030")
     )
     (path "/00000000-0000-0000-0000-000065179612"
